File: pv1000re.kicad_sch (KiCad schematic)
At the start: 201 parts, among them J1 Conn_02x18_Row_Letter_First, J2 Mini-DIN-8, J3 Mini-DIN-8, J4 Conn_01x05, J5 Barrel_Jack, Q1 2SA733, Q2 2SA733, Q3 2SA733, Q4 2SC945, Q5 2SC945, Q6 2SC945, Q7 2SC945, SW1 SW_SPST, U1 Z80CPU, U10 LM7805_TO220, U11 AN6040, U12 L7809, U13 D65010G031, U2 74LS04, U3 74LS74, U4 74LS163, U5 74LS74, U6 74LS32, U7 74LS07, U8 74LS05, U9 D4016, Y1 17.897727MHz

Commit message: Power and ground pins on ASIC. rename "ula" to "asic". Map pins on asic for joysticks to logical addresses
Connections:
- net ULAp11 is gone; now on net GND: R25.2, U13.11 (GND)
- net GND: now also U13.27 (GND)
- net VCC: now also U13.58 (VCC)
- net GPIb3: now reaches C18.1, J3.2, R39.1, RN7.5 (R4), TP33.1
- net GPIb2: now reaches C15.2, J3.7, R38.1, RN7.3 (R2), TP35.1
- net GPIb0: now reaches C16.2, J2.7, R40.1, RN7.2 (R1), TP36.1
- net gpo52 renamed GPOb3
- net gpo53_1 renamed GPOb2_1
- net gpo53_2 renamed GPOb2_2
- net gpo54 renamed GPOb1
- net gpo55 renamed GPOb0
- net ulaBlue renamed asicBlue
- net ulaGreen renamed asicGreen
- net ulaRed renamed asicRed
- net ulaSqF8 renamed asicSqF8
- net ulaSqF9 renamed asicSqF9
- net ulaSqFA renamed asicSqFA
- net ~{ulaColorburst} renamed ~{asicColorburst}
- net ~{ulaCsync} renamed ~{asicCsync}
Other:
- note added: "Schematic reverse-engineered by Lidnariq 2023 Copyright renounced: redistribute as Public Domain, CC0, or MIT-0 Attribution appreciated but not required"
- note removed: "Schematic reverse-engineered by Lidnariq 2023 Schematics are deemed not copyrightable in the US None-the-less, please give attribution if you use this"
- moved on the sheet: R28, U13, U8A
